File: E1600T/E1600T.kicad_sch (KiCad schematic)
At the start: 11 parts, among them J2 SWD, P1 Sensors, P6 Control board, P7 Boundary wire sensor, P8 Boundary wire sensor, P9 Rain Sensor, U11 R-Motor, U12 L-Motor, U6 STM32F103VCTx, U7 LMV358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

Commit message: Schematic updates
Parts:
- added J1: USB_B_Mini, Connector_USB:USB_Micro-B_Wuerth_614105150721_Vertical_CircularHoles, symbol Connector:USB_B_Mini
- added P13: Run Motor R, symbol Connector_Generic:Conn_01x02
- added P14: Run Motor L, symbol Connector_Generic:Conn_01x02
- added P2: Cutting Motor, symbol Connector_Generic:Conn_01x02
- added R13, R14, R15, R16, R17: R, symbol pspice:R
Connections:
- net GND: now also J1.5 (GND), R17.2
- net at U6.68 (PA9): now also R13.1, R17.1
- net at U6.69 (PA10): now also R14.1
- net at U6.70 (PA11): now also R15.1
- net at U6.71 (PA12): now also R16.2
- net at U11.13 (OUT3), U11.3 (OUT2): now also P13.1 (Pin_1)
- net at U11.14 (OUT4), U11.2 (OUT1): now also P13.2 (Pin_2)
- net at U12.13 (OUT3), U12.3 (OUT2): now also P14.1 (Pin_1)
- net at U12.14 (OUT4), U12.2 (OUT1): now also P14.2 (Pin_2)
- new net: J1.2 (D-), R15.2
- new net: J1.3 (D+), R14.2, R16.1
- new net: J1.1 (VBUS), R13.2
Other:
- moved on the sheet: J2, P6, U9F

Commit message: Added photos
Parts:
- added K1: Cutter relay, symbol Relay:IM47
Changed lines of the file:
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@@
-    (stroke (width 0) (type default) (color 0 0 0 0))
-  )
-  (wire (pts (xy 72.39 59.69) (xy 72.39 124.46))
     (stroke (width 0) (type default) (color 0 0 0 0))
   )
@@
     (stroke (width 0) (type default) (color 0 0 0 0))
   )
-  (wire (pts (xy 72.39 124.46) (xy 76.2 116.84))
-    (stroke (width 0) (type default) (color 0 0 0 0))
-  )
   (wire (pts (xy 259.08 130.81) (xy 255.27 130.81))
     (stroke (width 0) (type default) (color 0 0 0 0))
@@
     (stroke (width 0) (type default) (color 0 0 0 0))
   )
+  (wire (pts (xy 72.39 59.69) (xy 72.39 116.84))
+    (stroke (width 0) (type default) (color 0 0 0 0))
+  )
   (wire (pts (xy 161.29 87.63) (xy 161.29 99.06))
     (stroke (width 0) (type default) (color 0 0 0 0))
@@
   )
   (wire (pts (xy 44.45 78.74) (xy 44.45 76.2))
+    (stroke (width 0) (type default) (color 0 0 0 0))
+  )
+  (wire (pts (xy 72.39 116.84) (xy 76.2 116.84))
     (stroke (width 0) (type default) (color 0 0 0 0))
   )
@@
     (pin "1")
   )
+  (symbol (lib_id "Relay:IM47") (at 240.03 100.33 0) (unit 1)
+    (in_bom yes) (on_board yes) (fields_autoplaced)
+    (property "Reference" "K1" (id 0) (at 256.54 99.0599 0)
+      (effects (font (size 1.27 1.27)) (justify left))
+    )
+    (property "Value" "Cutter relay" (id 1) (at 256.54 101.5999 0)
+      (effects (font (size 1.27 1.27)) (justify left))
+    )
+    (property "Footprint" "" (id 2) (at 240.03 100.33 0)
+      (effects (font (size 1.27 1.27)) hide)
+    )
+    (property "Datasheet" "http://www.te.com/commerce/DocumentDelivery/DDEController?Action=srchrtrv&DocNm=108-98001&DocType=SS&DocLang=EN" (id 3) (at 240.03 100.33 0)
+      (effects (font (size 1.27 1.27)) hide)
+    )
+    (pin "7")
+    (pin "3")
+    (pin "5")
+    (pin "1")
+    (pin "2")
+    (pin "6")
+    (pin "4")
+    (pin "8")
+  )
   (symbol (lib_id "74xx:74HC14") (at 207.01 59.69 0) (unit 6)
     (in_bom yes) (on_board yes) (fields_autoplaced)
@@
       (reference "J2") (unit 1) (value "SWD") (footprint "")
     )
+    (path "/e6eb649b-ceac-4b1c-a2c4-1c23b899a3c9"
+      (reference "K1") (unit 1) (value "Cutter relay") (footprint "")
+    )
     (path "/59439b20-9695-4818-94e8-edd7ad7ffa07"
